File: kvm-compute-cluster-led-indicator.sch (KiCad schematic (older format))
At the start: 26 parts, among them J1 TE_1-1734248-5_FLEX, U1 PCA9685BS,118

Commit message: Add OSHW Logo
Parts:
- added N1: antmicro_logo, antmicro-footprints:antmicro-logo_scaled_15mm_silk, symbol antmicroMechanicalParts:antmicro_logo
- added N2: oshw_logo, antmicro-footprints:OSHW-Logo_5.7x6mm_SilkScreen, symbol antmicroMechanicalParts:oshw_logo
Changed lines of the file:
@@
 Wire Wire Line
 	4750 2525 4750 2300
+$Comp
+L antmicroMechanicalParts:antmicro_logo N1
+U 1 1 603AD97C
+P 5900 7350
+F 0 "N1" H 6114 7443 50  0000 L CNN
+F 1 "antmicro_logo" H 6114 7352 50  0000 L CNN
+F 2 "antmicro-footprints:antmicro-logo_scaled_15mm_silk" H 5800 7600 50  0001 C CNN
+F 3 "" H 5900 7700 50  0001 C CNN
+	1    5900 7350
+	1    0    0    -1
+$EndComp
+$Comp
+L antmicroMechanicalParts:oshw_logo N2
+U 1 1 603B0192
+P 5050 7300
+F 0 "N2" H 5244 7303 50  0000 L CNN
+F 1 "oshw_logo" H 5244 7212 50  0000 L CNN
+F 2 "antmicro-footprints:OSHW-Logo_5.7x6mm_SilkScreen" H 5070 7060 50  0001 C CNN
+F 3 "" H 5050 7300 50  0001 C CNN
+	1    5050 7300
+	1    0    0    -1
+$EndComp
 $EndSCHEMATC

Commit message: Add 0R DNP resistor at ~OE pin
Parts:
- added R19: R_0R_0402, antmicro-footprints:0402-res, symbol antmicroResistors0402:R_0R_0402
Connections:
- wire segments 109 -> 112
Changed lines of the file:
@@
+	1    0    0    -1
+$EndComp
+$Comp
+L antmicroResistors0402:R_0R_0402 R19
+U 1 1 603FD960
+P 3325 3500
+F 0 "R19" V 3234 3570 60  0000 L CNN
+F 1 "R_0R_0402" H 3325 3350 60  0001 C CNN
+F 2 "antmicro-footprints:0402-res" H 3525 3700 60  0001 L CNN
+F 3 "" H 3325 3500 50  0001 C CNN
+F 4 "PANASONIC" H 3525 3900 60  0001 L CNN "Manufacturer"
+F 5 "ERJ2GE0R00X" H 3525 3800 60  0001 L CNN "MPN"
+F 6 "0R" V 3332 3570 50  0000 L CNN "Val"
+F 7 "DNP" V 3423 3570 50  0000 L CNN "DNP"
+	1    3325 3500
+	0    1    1    0
+$EndComp
+Wire Wire Line
+	3525 3275 3325 3275
+Wire Wire Line
+	3325 3275 3325 3350
+Connection ~ 3525 3275
+Wire Wire Line
+	3325 3650 3325 3800
+$Comp
+L power:GND #PWR0109
+U 1 1 60412CFF
+P 3325 3800
+F 0 "#PWR0109" H 3325 3550 50  0001 C CNN
+F 1 "GND" H 3330 3627 50  0000 C CNN
+F 2 "" H 3325 3800 50  0001 C CNN
+F 3 "" H 3325 3800 50  0001 C CNN
+	1    3325 3800
 	1    0    0    -1
 $EndComp

Commit message: Add local libraries
Parts:
- C1: footprint antmicro-footprints:0402-cap -> kvm-compute-cluster-led-indicator-footprints:0402-cap; symbol antmicroCapacitors0402:C_100n_0402 -> kvm-compute-cluster-led-indicator:C_100n_0402
- D1, D2, D3, D4, D5: footprint antmicro-footprints:LED_Dual0603 -> kvm-compute-cluster-led-indicator-footprints:LED_Dual0603; symbol antmicroLEDIndicationDiscrete:LTST-C19HE1WT -> kvm-compute-cluster-led-indicator:LTST-C19HE1WT
- J1: footprint antmicro-footprints:TE_1-1734248-5_FLEX -> kvm-compute-cluster-led-indicator-footprints:TE_1-1734248-5_FLEX; symbol antmicroFCCConnectors:TE_1-1734248-5_FLEX -> kvm-compute-cluster-led-indicator:TE_1-1734248-5_FLEX
- N1: footprint antmicro-footprints:antmicro-logo_scaled_15mm_silk -> kvm-compute-cluster-led-indicator-footprints:antmicro-logo_scaled_15mm_silk; symbol antmicroMechanicalParts:antmicro_logo -> kvm-compute-cluster-led-indicator:antmicro_logo
- N2: footprint antmicro-footprints:OSHW-Logo_5.7x6mm_SilkScreen -> kvm-compute-cluster-led-indicator-footprints:OSHW-Logo_5.7x6mm_SilkScreen; symbol antmicroMechanicalParts:oshw_logo -> kvm-compute-cluster-led-indicator:oshw_logo
- R1: footprint antmicro-footprints:0402-res -> kvm-compute-cluster-led-indicator-footprints:0402-res; symbol antmicroResistors0402:R_10k_0402 -> kvm-compute-cluster-led-indicator:R_10k_0402
- R10, R13, R16, R2, R5: footprint antmicro-footprints:0402-res -> kvm-compute-cluster-led-indicator-footprints:0402-res; symbol antmicroResistors0402:R_100R_0402 -> kvm-compute-cluster-led-indicator:R_100R_0402
- R11, R12, R14, R15, R17, R18, R3, R4, R6, R9: footprint antmicro-footprints:0402-res -> kvm-compute-cluster-led-indicator-footprints:0402-res; symbol antmicroResistors0402:R_49R9_0402 -> kvm-compute-cluster-led-indicator:R_49R9_0402
- R19: footprint antmicro-footprints:0402-res -> kvm-compute-cluster-led-indicator-footprints:0402-res; symbol antmicroResistors0402:R_0R_0402 -> kvm-compute-cluster-led-indicator:R_0R_0402
- R7, R8: footprint antmicro-footprints:0402-res -> kvm-compute-cluster-led-indicator-footprints:0402-res; symbol antmicroResistors0402:R_4k7_0402 -> kvm-compute-cluster-led-indicator:R_4k7_0402
- U1: footprint antmicro-footprints:QFN-28_6x6mm_P0.65mm -> kvm-compute-cluster-led-indicator-footprints:QFN-28_6x6mm_P0.65mm; symbol antmicroInterfaceIOExpanders:PCA9685BS,118 -> kvm-compute-cluster-led-indicator:PCA9685BS,118
