File: rpi-compute-cluster-led-indicator.kicad_pcb (KiCad board)
At the start: 2 copper layers, 70.3 x 35.6 mm, 29 parts, among them J1 TE_1-1734248-5_FLEX, U1 PCA9685BS,118

Commit message: Update naming convention
Parts:
- C1: footprint kvm-compute-cluster-led-indicator-footprints:0402-cap -> rpi-compute-cluster-led-indicator-footprints:0402-cap
- D1, D2, D3, D4, D5: footprint kvm-compute-cluster-led-indicator-footprints:LED_Dual0603 -> rpi-compute-cluster-led-indicator-footprints:LED_Dual0603
- J1: footprint kvm-compute-cluster-led-indicator-footprints:TE_1-1734248-5_FLEX -> rpi-compute-cluster-led-indicator-footprints:TE_1-1734248-5_FLEX
- N1: footprint kvm-compute-cluster-led-indicator-footprints:antmicro-logo_scaled_15mm_silk -> rpi-compute-cluster-led-indicator-footprints:antmicro-logo_scaled_15mm_silk
- N2: footprint kvm-compute-cluster-led-indicator-footprints:OSHW-Logo_5.7x6mm_SilkScreen -> rpi-compute-cluster-led-indicator-footprints:OSHW-Logo_5.7x6mm_SilkScreen
- R1, R10, R11, R12, R13, R14, R15, R16, R17, R18, R19, R2, R3, R4, R5, R6, R7, R8, R9: footprint kvm-compute-cluster-led-indicator-footprints:0402-res -> rpi-compute-cluster-led-indicator-footprints:0402-res
- U1: footprint kvm-compute-cluster-led-indicator-footprints:QFN-28_6x6mm_P0.65mm -> rpi-compute-cluster-led-indicator-footprints:QFN-28_6x6mm_P0.65mm

Commit message: Assign revision 1.1.0
Other:
- board text added: "Rpi Compute Cluster LED indicator Rev.1.1.0"
- board text removed: "KVM cluster LED indicator Rev.1.0.1 10/2021"
