File: rpi-led-flex-board.sch (KiCad schematic (older format))
At the start: 29 parts, among them J1 TE_1-1734248-5_FLEX, U1 PCA9685BS,118

Commit message: Update naming convention
Parts:
- C1: footprint rpi-compute-cluster-led-indicator-footprints:0402-cap -> rpi-led-flex-board-footprints:0402-cap; symbol rpi-compute-cluster-led-indicator:C_100n_0402 -> rpi-led-flex-board:C_100n_0402
- D1, D2, D3, D4, D5: footprint rpi-compute-cluster-led-indicator-footprints:LED_Dual0603 -> rpi-led-flex-board-footprints:LED_Dual0603; symbol rpi-compute-cluster-led-indicator:LTST-C19HE1WT -> rpi-led-flex-board:LTST-C19HE1WT
- J1: footprint rpi-compute-cluster-led-indicator-footprints:TE_1-1734248-5_FLEX -> rpi-led-flex-board-footprints:TE_1-1734248-5_FLEX; symbol rpi-compute-cluster-led-indicator:TE_1-1734248-5_FLEX -> rpi-led-flex-board:TE_1-1734248-5_FLEX
- N1: footprint rpi-compute-cluster-led-indicator-footprints:antmicro-logo_scaled_15mm_silk -> rpi-led-flex-board-footprints:antmicro-logo_scaled_15mm_silk; symbol rpi-compute-cluster-led-indicator:antmicro_logo -> rpi-led-flex-board:antmicro_logo
- N2: footprint rpi-compute-cluster-led-indicator-footprints:OSHW-Logo_5.7x6mm_SilkScreen -> rpi-led-flex-board-footprints:OSHW-Logo_5.7x6mm_SilkScreen; symbol rpi-compute-cluster-led-indicator:oshw_logo -> rpi-led-flex-board:oshw_logo
- R1: footprint rpi-compute-cluster-led-indicator-footprints:0402-res -> rpi-led-flex-board-footprints:0402-res; symbol rpi-compute-cluster-led-indicator:R_10k_0402 -> rpi-led-flex-board:R_10k_0402
- R10, R13, R16, R2, R5: footprint rpi-compute-cluster-led-indicator-footprints:0402-res -> rpi-led-flex-board-footprints:0402-res; symbol rpi-compute-cluster-led-indicator:R_100R_0402 -> rpi-led-flex-board:R_100R_0402
- R11, R12, R14, R15, R17, R18, R3, R4, R6, R9: footprint rpi-compute-cluster-led-indicator-footprints:0402-res -> rpi-led-flex-board-footprints:0402-res; symbol rpi-compute-cluster-led-indicator:R_49R9_0402 -> rpi-led-flex-board:R_49R9_0402
- R19: footprint rpi-compute-cluster-led-indicator-footprints:0402-res -> rpi-led-flex-board-footprints:0402-res; symbol rpi-compute-cluster-led-indicator:R_0R_0402 -> rpi-led-flex-board:R_0R_0402
- R7, R8: footprint rpi-compute-cluster-led-indicator-footprints:0402-res -> rpi-led-flex-board-footprints:0402-res; symbol rpi-compute-cluster-led-indicator:R_4k7_0402 -> rpi-led-flex-board:R_4k7_0402
- U1: footprint rpi-compute-cluster-led-indicator-footprints:QFN-28_6x6mm_P0.65mm -> rpi-led-flex-board-footprints:QFN-28_6x6mm_P0.65mm; symbol rpi-compute-cluster-led-indicator:PCA9685BS,118 -> rpi-led-flex-board:PCA9685BS,118
